Commit message: Bug Solved

File: urdf/car.urdf.xacro (robot description, xacro)
@@ -78,5 +78,5 @@
 	</link>
 	<joint name="joint_right_wheel_chassis" type="continuous">
-		<origin rpy="0 0 0" xyz="-0.05 ${b1/2} 0"/>
+		<origin rpy="0 0 0" xyz="-0.05 -${b1/2} 0"/>
 		<child link="right_wheel"/>
 		<parent link="chassis"/>
@@ -106,5 +106,5 @@
 	</link>
 	<joint name="joint_left_wheel_chassis" type="continuous">
-		<origin rpy="0 0 0" xyz="-0.05 -${b1/2} 0"/>
+		<origin rpy="0 0 0" xyz="-0.05 ${b1/2} 0"/>
 		<child link="left_wheel"/>
 		<parent link="chassis"/>
@@ -141,4 +141,10 @@
 		<parent link="chassis"/>
 	</joint>
+	<link name="kinect_link" />
+	<joint name="joint_kinect_link" type="continuous">
+		<origin rpy="-1.5707 0 -1.5707" xyz="${l1/2} 0 ${h1/2+hk/2}"/>
+		<child link="kinect_link"/>
+		<parent link="chassis"/>
+	</joint>
 <xacro:include filename="$(find navros_pkg)/urdf/gazebo_plugins.urdf.xacro" />
 </robot>

File: urdf/gazebo_plugins.urdf.xacro (robot description, xacro)
@@ -57,5 +57,5 @@
 		        <updateRate>10.0</updateRate>
 		        <cameraName>kinect</cameraName>
-		        <frameName>joint_kinect_chassis</frameName>
+		        <frameName>kinect_link</frameName>
 		    <imageTopicName>rgb/image_raw</imageTopicName>
 		    <depthImageTopicName>depth/image_raw</depthImageTopicName>

Commit message: Update

File: urdf/car.urdf.xacro (robot description, xacro)
@@ -142,5 +142,5 @@
 	</joint>
 	<link name="kinect_link" />
-	<joint name="joint_kinect_link" type="continuous">
+	<joint name="joint_kinect_link" type="fixed">
 		<origin rpy="-1.5707 0 -1.5707" xyz="${l1/2} 0 ${h1/2+hk/2}"/>
 		<child link="kinect_link"/>
